File: project-hw-usbc-mux-demux.kicad_pcb (KiCad board)
At the start: 4 copper layers, 40 x 30 mm, 24 parts, among them J1 Amphenol_12402012E212A, J2 Amphenol_12402012E212A, J3 Amphenol_12402012E212A, J4 Conn_01x04_Pin, Q1 Q_Toshiba_SSM3J328R, Q2 Q_Toshiba_SSM3J328R, U1 LMR516x5, U2 FUSB303BTMX

Commit message: Add assembly file
Parts:
- Q1, Q2: value Q_Toshiba_SSM3J328R -> SSM3J328R
Changed lines of the file:
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@@
 		)
 		(property "Value" "0.1uF"
-			(at 0 1.43 90)
+			(at 3.5 0 90)
 			(layer "F.Fab")
 			(effects
@@
 		)
 		(property "Value" "10k"
-			(at 0 1.43 90)
+			(at -3 0 90)
 			(layer "F.Fab")
 			(effects
@@
 			)
 		)
-		(property "Value" "Q_Toshiba_SSM3J328R"
-			(at 0 3 90)
+		(property "Value" "SSM3J328R"
+			(at 2 -2 0)
 			(layer "F.Fab")
 			(effects
@@
 		(tags "USB C Type-C Receptacle SMD USB 2.0 16P 16C USB4105-15-A USB4105-15-A-060 USB4105-15-A-120 USB4105-GF-A USB4105-GF-A-060 USB4105-GF-A-120 12402012E212A")
 		(property "Reference" "J1"
-			(at 0 -6 270)
+			(at 0 -6 -90)
 			(unlocked yes)
 			(layer "F.SilkS")
@@
 		)
 		(property "Value" "Amphenol_12402012E212A"
-			(at 0 5 -90)
+			(at -7 -6 0)
 			(unlocked yes)
 			(layer "F.Fab")
@@
 		)
 		(property "Value" "LED_Small"
-			(at 0 1.43 90)
+			(at 0 1.5 90)
 			(layer "F.Fab")
+			(hide yes)
 			(effects
 				(font
@@
 		)
 		(property "Value" "1k"
-			(at 0 1.43 90)
+			(at -0.5 -1.5 90)
 			(layer "F.Fab")
 			(effects
@@
 			)
 		)
-		(property "Value" "Q_Toshiba_SSM3J328R"
-			(at 0 3 90)
+		(property "Value" "SSM3J328R"
+			(at -6.5 -1 270)
 			(layer "F.Fab")
+			(hide yes)
 			(effects
 				(font
@@
 		)
 		(property "Value" "10k"
-			(at 0 1.43 90)
+			(at 0.5 1.43 90)
 			(layer "F.Fab")
 			(effects
@@
 			(unlocked yes)
 			(layer "F.Fab")
+			(hide yes)
 			(effects
 				(font
@@
 		)
 		(property "Value" "22uF 16V"
-			(at 0 2.3 90)
+			(at 3 -2 180)
 			(layer "F.Fab")
 			(effects
@@
 		)
 		(property "Value" "52.3k"
-			(at 0 1.43 90)
+			(at -3.5 0 90)
 			(layer "F.Fab")
 			(effects
@@
 		)
 		(property "Value" "5.1V"
-			(at 0 2 0)
+			(at 3.5 0 0)
 			(layer "F.Fab")
 			(effects
@@
 		)
 		(fp_text user "${REFERENCE}"
-			(at 0 -2 0)
+			(at -0.5 -1.5 0)
 			(layer "F.Fab")
+			(hide yes)
 			(effects
 				(font
@@
 		)
 		(property "Value" "10k"
-			(at 0 1.43 90)
+			(at 3 0 90)
 			(layer "F.Fab")
 			(effects
@@
 		(tags "Texas X2QFN NoLead")
 		(property "Reference" "U2"
-			(at 0 -3 360)
+			(at 0 -3 0)
 			(layer "F.SilkS")
 			(hide yes)
@@
 		)
 		(property "Value" "FUSB303BTMX"
-			(at 0 3 360)
+			(at 1.5 -2.5 0)
 			(layer "F.Fab")
 			(effects
@@
 		)
 		(property "Footprint" "QFN:Texas_X2QFN-12_1.6x1.6mm_P0.4mm"
-			(at 0 0 360)
+			(at 0 0 0)
 			(layer "F.Fab")
 			(hide yes)
@@
 		)
 		(property "Datasheet" "https://www.onsemi.com/pdf/datasheet/fusb303b-d.pdf"
-			(at 0 0 360)
+			(at 0 0 0)
 			(layer "F.Fab")
 			(hide yes)
@@
 		)
 		(property "Description" "USB Type-C port controller with I2C and GPIO control, X2QFN-12"
-			(at 0 0 360)
+			(at 0 0 0)
 			(layer "F.Fab")
 			(hide yes)
@@
 		)
 		(fp_text user "${REFERENCE}"
-			(at 0 0 360)
+			(at 0 0 0)
 			(layer "F.Fab")
 			(effects
@@
 			(at 0 1.55 0)
 			(layer "F.Fab")
+			(hide yes)
 			(effects
 				(font
@@
 		)
 		(property "Value" "10k"
-			(at 0 1.43 90)
+			(at 0 -1.5 90)
 			(layer "F.Fab")
 			(effects
@@
 		)
 		(property "Value" "22uF 16V"
-			(at 0 2.3 90)
+			(at 0 -2.5 90)
 			(layer "F.Fab")
+			(hide yes)
 			(effects
 				(font
@@
 		)
 		(property "Value" "100k"
-			(at 0 1.43 0)
+			(at 3.5 0 0)
 			(layer "F.Fab")
 			(effects
@@
 			(unlocked yes)
 			(layer "F.Fab")
+			(hide yes)
 			(effects
 				(font
@@
 			(at 0 9.95 90)
 			(layer "F.Fab")
+			(hide yes)
 			(effects
 				(font
@@
 		)
 		(property "Value" "LMR516x5"
-			(at 0 3 0)
+			(at -5.5 -2.5 90)
 			(layer "F.Fab")
 			(effects
@@
 		)
 		(property "Value" "6.8uH"
-			(at 0 4 0)
+			(at 0 -4 0)
 			(unlocked yes)
 			(layer "F.Fab")
@@
 		(polygon
 			(pts
-				(xy 38 43.5) (xy 39.5 43.5) (xy 39.5 43.5) (xy 43.5 43.5) (xy 43.5 36) (xy 38 36)
+				(xy 38 43.5) (xy 39.5 43.5) (xy 43.5 43.5) (xy 43.5 36) (xy 38 36)
 			)
 		)
